Commit message: pcl

File: crane_x7_description/urdf/crane_x7_mounting_plate.xacro (robot description, xacro)
@@ -32,4 +32,76 @@
       <material>Gazebo/Black</material>
     </gazebo>
+    <link name="real_link_optical_frame" />
+    <link name="real_depth_frame"/>
+    <link name="real_link">
+      <visual>
+        <geometry>
+          <box size="0.025 0.090 0.025"/>
+        </geometry>
+        <material name="green"/>
+      </visual>
+      <collision>
+        <geometry>
+          <box size="0.025 0.090 0.025"/>
+        </geometry>
+      </collision>
+      <inertial>
+        <origin xyz="0 0 0" rpy="0 0 0"/>
+        <mass value="1"/>
+        <inertia
+          ixx="1.04e-4" ixy="0.0" ixz="0.0"
+          iyy="7.27e-4" iyz="0.0"
+          izz="1.04e-4"/>
+        </inertial>
+    </link>
+    <joint name="real_base_joint" type="fixed">
+      <origin xyz="0.3 0.0 0.7" rpy="0 1.57 0"/>
+      <parent link="base_link"/>
+      <child link="real_link_optical_frame"/>
+    </joint>
+    <joint name="real_depth_joint" type="fixed">
+        <origin xyz="0 0 0" rpy="${-M_PI/2} 0 ${-M_PI/2}" />
+      <parent link="real_link_optical_frame" />
+      <child link="real_depth_frame" />
+    </joint>
+    <joint name="real_joint" type="fixed">
+      <origin xyz="0 0 0" rpy="0 0 0"/>
+      <parent link="real_link_optical_frame"/>
+      <child link="real_link"/>
+    </joint>
+    <gazebo reference="real_link">
+      <sensor type="depth" name="real_ir_sensor">
+        <always_on>true</always_on>
+        <update_rate>40.0</update_rate>
+        <camera>
+          <horizontal_fov>${91.2*M_PI/180.0}</horizontal_fov>
+          <image>
+            <format>R8G8B8</format>
+            <width>1280</width>
+            <height>720</height>
+          </image>
+          <clip>
+            <near>0.2</near>
+            <far>10.0</far>
+          </clip>
+        </camera>
+        <plugin name="real_link_controller" filename="libgazebo_ros_openni_kinect.so">
+          <alwaysOn>true</alwaysOn>
+          <updateRate>1.0</updateRate>
+          <cameraName>camera</cameraName>
+          <depthImageTopicName>/camera/depth_registered/image_raw</depthImageTopicName>
+          <depthImageCameraInfoTopicName>/camera/depth/camera_info</depthImageCameraInfoTopicName>
+          <pointCloudTopicName>/camera/depth_registered/points</pointCloudTopicName>
+          <frameName>real_depth_frame</frameName>
+          <pointCloudCutoff>0.5</pointCloudCutoff>
+          <distortionK1>0.00000001</distortionK1>
+          <distortionK2>0.00000001</distortionK2>
+          <distortionK3>0.00000001</distortionK3>
+          <distortionT1>0.00000001</distortionT1>
+          <distortionT2>0.00000001</distortionT2>
+        </plugin>
+      </sensor>
+      <material value="Gazebo/Blue" />
+    </gazebo>
   </xacro:macro>
 </robot>

Commit message: cameratuketa

File: crane_x7_description/urdf/crane_x7_mounting_plate.xacro (robot description, xacro)
@@ -32,76 +32,4 @@
       <material>Gazebo/Black</material>
     </gazebo>
-    <link name="real_link_optical_frame" />
-    <link name="real_depth_frame"/>
-    <link name="real_link">
-      <visual>
-        <geometry>
-          <box size="0.025 0.090 0.025"/>
-        </geometry>
-        <material name="green"/>
-      </visual>
-      <collision>
-        <geometry>
-          <box size="0.025 0.090 0.025"/>
-        </geometry>
-      </collision>
-      <inertial>
-        <origin xyz="0 0 0" rpy="0 0 0"/>
-        <mass value="1"/>
-        <inertia
-          ixx="1.04e-4" ixy="0.0" ixz="0.0"
-          iyy="7.27e-4" iyz="0.0"
-          izz="1.04e-4"/>
-        </inertial>
-    </link>
-    <joint name="real_base_joint" type="fixed">
-      <origin xyz="0.3 0.0 0.7" rpy="0 1.57 0"/>
-      <parent link="base_link"/>
-      <child link="real_link_optical_frame"/>
-    </joint>
-    <joint name="real_depth_joint" type="fixed">
-        <origin xyz="0 0 0" rpy="${-M_PI/2} 0 ${-M_PI/2}" />
-      <parent link="real_link_optical_frame" />
-      <child link="real_depth_frame" />
-    </joint>
-    <joint name="real_joint" type="fixed">
-      <origin xyz="0 0 0" rpy="0 0 0"/>
-      <parent link="real_link_optical_frame"/>
-      <child link="real_link"/>
-    </joint>
-    <gazebo reference="real_link">
-      <sensor type="depth" name="real_ir_sensor">
-        <always_on>true</always_on>
-        <update_rate>40.0</update_rate>
-        <camera>
-          <horizontal_fov>${91.2*M_PI/180.0}</horizontal_fov>
-          <image>
-            <format>R8G8B8</format>
-            <width>1280</width>
-            <height>720</height>
-          </image>
-          <clip>
-            <near>0.2</near>
-            <far>10.0</far>
-          </clip>
-        </camera>
-        <plugin name="real_link_controller" filename="libgazebo_ros_openni_kinect.so">
-          <alwaysOn>true</alwaysOn>
-          <updateRate>1.0</updateRate>
-          <cameraName>camera</cameraName>
-          <depthImageTopicName>/camera/depth_registered/image_raw</depthImageTopicName>
-          <depthImageCameraInfoTopicName>/camera/depth/camera_info</depthImageCameraInfoTopicName>
-          <pointCloudTopicName>/camera/depth_registered/points</pointCloudTopicName>
-          <frameName>real_depth_frame</frameName>
-          <pointCloudCutoff>0.5</pointCloudCutoff>
-          <distortionK1>0.00000001</distortionK1>
-          <distortionK2>0.00000001</distortionK2>
-          <distortionK3>0.00000001</distortionK3>
-          <distortionT1>0.00000001</distortionT1>
-          <distortionT2>0.00000001</distortionT2>
-        </plugin>
-      </sensor>
-      <material value="Gazebo/Blue" />
-    </gazebo>
   </xacro:macro>
 </robot>
