Commit message: comitto

File: crane_x7_description/urdf/camera.urdf (robot description, URDF)
Before this commit: robot camera, 3 links, 3 joints
Joints:
- joint real_base_joint: origin xyz=0 0.1 0 rpy=0 1.57 0 -> xyz=0 0.05 0 rpy=0 -1.570795 -1.570795
- joint real_depth_joint: origin xyz=0 0 0 rpy=-1.570795 0 -1.570795 -> xyz=0 0 0 rpy=0 0 0

Commit message: aa

File: crane_x7_description/urdf/camera.urdf (robot description, URDF)
Before this commit: robot camera, 3 links, 3 joints
Links:
- link real_link: geometry visual box size=0.025 0.090 0.025

File: crane_x7_description/urdf/crane_x7.urdf.xacro (robot description, xacro)
@@ -22,14 +22,14 @@
        right-handed robots. -->
   <crane_x7 parent="base_link"
-              base_color="white"
-              shoulder_color="blue"
-              shoulder_joint_cover_color="white"
-              upper_arm_upper_color="blue"
-              upper_arm_lower_color="blue"
-              elbow_joint_cover_color="white"
-              lower_arm_upper_color="blue"
+              base_color="red"
+              shoulder_color="white"
+              shoulder_joint_cover_color="red"
+              upper_arm_upper_color="white"
+              upper_arm_lower_color="white"
+              elbow_joint_cover_color="red"
+              lower_arm_upper_color="white"
               lower_arm_lower_color="white"
               wrist_color="white"
-              hand_color="white"
+              hand_color="red"
               joints_vlimit="4.81710873"
               shoulder_llimit="-2.97132"

File: crane_x7_description/urdf/crane_x7.xacro (robot description, xacro)
@@ -4,5 +4,5 @@
   <xacro:include filename="$(find crane_x7_description)/urdf/crane_x7_arm.xacro"/>
   <xacro:include filename="$(find crane_x7_description)/urdf/crane_x7_wide_two_finger_gripper.xacro"/>
-  <xacro:include filename="$(find crane_x7_description)/urdf/camera.urdf"/>
+  <!--<xacro:include filename="$(find crane_x7_description)/urdf/camera.urdf"/>-->
   <material name="black">
     <color rgba="0.2 0.2 0.2 1.0"/>

Commit message: torima

File: crane_x7_description/urdf/camera.urdf (robot description, URDF)
Before this commit: robot camera, 3 links, 3 joints
Links:
- link real_link: geometry collision box size=0.0001 0.0001 0.0001; visual box size=0.025 0.090 0.025

File: crane_x7_description/urdf/crane_x7.xacro (robot description, xacro)
@@ -4,5 +4,5 @@
   <xacro:include filename="$(find crane_x7_description)/urdf/crane_x7_arm.xacro"/>
   <xacro:include filename="$(find crane_x7_description)/urdf/crane_x7_wide_two_finger_gripper.xacro"/>
-  <!--<xacro:include filename="$(find crane_x7_description)/urdf/camera.urdf"/>-->
+  <xacro:include filename="$(find crane_x7_description)/urdf/camera.urdf"/>
   <material name="black">
     <color rgba="0.2 0.2 0.2 1.0"/>
